File: Little PA V2.kicad_sch (KiCad schematic)
At the start: 90 parts, among them IC1 SX1255, J1 U.FL, J2 U.FL, J3 RPi, J4 WP, Q1 BSS84, U1 MCP1703Ax-330xxDB, U2 24LC256, U3 74LVC1G74DP_125, U4 TQP3M9036, U5 SRV05-4, X1 TA0655A, X2 TA2490A, Y1 38.4MHz

Commit message: Add files via upload
Parts:
- X1: now in the parts list
Changed lines of the file:
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@@
 	(title_block
 		(title "HAT little PA V2")
-		(date "2026-06-02")
+		(date "2026-09-28")
 		(rev "V2.0")
 		(company "Z32IT")
@@
 		(body_style 1)
 		(exclude_from_sim no)
-		(in_bom no)
+		(in_bom yes)
 		(on_board yes)
 		(in_pos_files yes)
